File: pcb/0.2/0.2.sch (EAGLE design)
At the start: 51 parts, among them Q1 FDS6699, Q2 FDS6699, U1 PIC18F26K20-E/SS, U2 UCC27211A, U4 INA-139, U5 INA-139, U6 INA-139, U7 R-78EXX, X1 8M

Commit message: Fixed: Output not turning on after low voltage shutdown
Parts:
- C10, C11, C12, C13, C14, C15, C18, C19, C2, C4, C5, C7, ICSP, LCD, Q7, R1, R13, R14, R15, R3, R4, R5, R6, R7, R8, R9, S1: PARTNO (none) -> *
- C16, C3, C8, C9: PARTNO (none) -> 35ZLH220MEFC8X11.5
- D1: PARTNO (none) -> SK54B-LTP
- F4: PARTNO (none) -> C1T 5
- H_UART: PARTNO (none) -> B3B-XH-A (LF)(SN)(P)
- L1: PARTNO (none) -> IHLP6767GZER330M11
- Q1, Q2: PARTNO (none) -> SI4128DY-T1-GE3
- Q3, Q4: PARTNO (none) -> BSH103,215
- Q5, Q6: PARTNO (none) -> FDS6681Z
- RS1, RS2, RS3: PARTNO (none) -> PMR25HZPFV2L00
- U1: PARTNO (none) -> PIC18F26K22-I/SS
- U2: PARTNO (none) -> UCC27211D
- U4, U5, U6: PARTNO (none) -> INA139NA/250
- U7: PARTNO (none) -> R-78E3.3-0.5
- X1: PARTNO (none) -> 7A-8.000MAAE-T
